File: enduro/enduro.kicad_sch (KiCad schematic)
At the start: 127 parts

Commit message: Snapshot 220425
- The Flipsky Antispark switch blew up on first usage, so I replaced it with an SSR connected to the antitheft lines. The system is always powered on (the current BMS doesn't have an 'off' switch) but you can't drive it anywhere, and the quiescent power usage is acceptably low.
- Moved the horn to the fork
- Wireless antitheft! There's a small 'bootstrap' battery (1S3P 18650.) It powers a 12V boost converter which runs a Solidremote 202U two-channel relay board. This listens for 'antitheft on/off' and 'BMS pulse' signals from the remote. AT On/Off is wired to the antitheft SSR.
- Added a 5V DCDC with three USB outputs. Its jobs are:
    1. Charge the bootstrap battery
    2. (later) run a USB panel socket for phone charging
    3. (later) power an internal body controller
- The bar cutoff/kill switch is now wired in series with the antitheft line, so BOTH the antitheft AND the cutoff must be deasserted to allow power to the motor.
- If the cutoff is open you can't tell if the antitheft is active, so I put a red LED ("AT LED") on the side to show when the antitheft is enabled or disabled.
- The brake light relay board didn't work as planned, so I replaced it with a soldered-in SSR.

I've been running this for a couple of months for daily commutes and it's comfy up to about 40mph. The limit right now is the hopelessly saggy UPP battery; it's limiting to about 50A at 60V (3kW; should be 16S = 67.2V.) I have two batteries in production (a 'high range' 18650 pack and a 'max current' SPIM pouch pack) and so should be able to test at higher power levels soon.
Parts:
- removed J? (x2): BNC, symbol Connector_Generic:Conn_01x03
- removed J?: Conn_01x02, symbol Connector_Generic:Conn_01x02
- removed SW?: SW_SPST, symbol Switch:SW_SPST
- added BT? (x2): Battery_Cell, symbol Device:Battery_Cell
- added BT?: 18650, symbol Device:Battery_Cell
- added D?: Antitheft disarmed (red), symbol Device:LED
- added J? (x3): Conn_01x02, symbol Connector_Generic:Conn_01x02
- added J?: Relay 1, symbol Connector_Generic:Conn_01x03
- added J? (x5): USB-A socket, symbol Connector_Generic:Conn_01x02
- added J? (x2): Tail lights, symbol Connector_Generic:Conn_01x03
- added J? (x3): AT LED, symbol Connector_Generic:Conn_01x02
- added J?: BMS BTN, symbol Connector_Generic:Conn_01x02
- added J?: Relay 2, symbol Connector_Generic:Conn_01x03
- added J?: AT CTRLR, symbol Connector:Screw_Terminal_01x01
- added J?: 1S BMS, symbol Connector_Generic:Conn_02x02_Odd_Even
- added J?: CUTOFF, symbol Connector_Generic:Conn_01x02
- added PS?: DROK 12V-5V Buck, Converter_DCDC:Converter_DCDC_Murata_MEE1SxxxxSC_THT, symbol Converter_DCDC:MEE1S0303SC
- added U?: S102S01, Package_SIP:SIP4_Sharp-SSR_P7.62mm_Straight, symbol Relay_SolidState:S102S01
- added U?: SSR, Package_SIP:SIP4_Sharp-SSR_P7.62mm_Straight, symbol Relay_SolidState:S102S01
- added U?: 12V_Boost, symbol enduro-libs:12V_Boost
Connections:
- net 12V (red): now also J?.3 (Pin_3); no longer J?.2 (Pin_2)
- net 84V: no longer J?.1 (Pin_1)
- net 84V (red?): no longer SW?.1 (A)
- net AUX (white): now also J?.2 (Pin_2), J?.2 (Pin_2), J?.3 (Pin_3), SW?.2 (B), J?.2 (Pin_2), J?.2 (Pin_2), J?.2 (Pin_2), U?.4
- net Brake12V (red): now also J?.1 (Pin_1); no longer J?.2 (Pin_2)
- net DRL (red): now also J?.2 (Pin_2), U?.3
- net EBK (red): now also J?.2 (Pin_2); no longer J?.1 (Pin_1)
- net Ignition (green): now also J?.1 (Pin_1); no longer J?.7 (Pin_7)
- net Cutoff1: no longer names the net of J?.1 (Pin_1)
- net Cutoff2: no longer names the net of J?.2 (Pin_2)
- removed net GND: J?.2 (Pin_2), J?.2 (Pin_2), J?.2 (Pin_2), J?.3 (Pin_3), SW?.2 (B)
- new net: J?.1 (Pin_1), J?.1 (Pin_1), J?.1 (Pin_1), PS?.4 (+Vout)
- new net: J?.2 (Pin_2), J?.2 (Pin_2), J?.2 (Pin_2), PS?.3 (-Vout)
- new net: J?.3 (Pin_3), U?.1
- new net: J?.2 (Pin_2), U?.2
- new net: J?.1 (Pin_1), U?. (VOUT-)
- new net: J?.2 (Pin_2), U?. (VOUT-)
- new net +12V: J?.1 (Pin_1), J?.1 (Pin_1), J?.1 (Pin_1), J?.2 (Pin_2), J?.2 (Pin_2)
- new net B+: BT?.1 (+), BT?.1 (+), BT?.1 (+), J?.1 (Pin_1)
- new net B-: BT?.2 (-), BT?.2 (-), BT?.2 (-), J?.3 (Pin_3)
- new net Brake12V (blue): J?.2 (Pin_2), J?.2 (Pin_2)
- new net NC: J?.1 (Pin_1), J?.1 (Pin_1)
- new net NO: J?.1 (Pin_1), J?.1 (Pin_1), J?.2 (Pin_2), J?.3 (Pin_3), J?.3 (Pin_3)
- new net OUT+: U?.1
- new net OUT-: U?.2
- new net P+: J?.2 (Pin_2), U?. (VOUT-)
- new net P-: J?.4 (Pin_4), U?. (VOUT-)
- new net Vbatt (red): J?.7 (Pin_7)
- no-connect marks 7 -> 10
Other:
- note added: "12V STANDBY"
- note added: "12VSB charger"
- note added: "Antitheft LED stays lit even if the cutoff is open. It's your reminder to lock the bike before walking away."
- note added: "Antitheft line to controller and CAv3"
- note added: "EBK has a weak 5V pullup. It pulls to GND when ebrake is engaged"
- note added: "Mounted in top case near the charge port"
- note added: "Not sure why Vbatt on CAv3 must not be connected, but if I power it, the system is always on. Powering CAv3 exclusively from orange (key return) line seems to be sufficient."
- note added: "Some of the wiring is bundled inside the remote case"
- note added: "TODO"
- note added: "TODO note down SSR part number"
- note added: "TODO remove flipsky"
- note added: "TODO replace with AS150"
- note added: "The 5V line only has about 10mA of source capacity at 84V and we use 5mA on the throttle. This SSR is supposed to use less than 5mA at 5V. Exceeding the CA5V current limit causes the screen to wash out and ADC reading to go bad."
- note added: "UP TO HERE CAV3 orange and Sabvoton ignition both go to bullet connector which connects back to SSR -OUT"
- note removed: "Brake Relay"
- note removed: "EBK pulls to GND when ebrake is engaged"
- note removed: "TODO check pin ordering for ebrake line"
- note removed: "TODO: this circuit is not working LED lights up but we don't see any switching on the output"
- note removed: "The two GNDs are isolated."
- note removed: "put a remote relay here somewhere inline with the cutoff"
- moved on the sheet: A?

Commit message: 5V conversion
- Remove the internal starter pack -- it kept running flat.
- Replace the remote receiver with a 5V version.
- Add a 5V standby DCDC which is always on.
- Add a switched 84V-5V DCDC which is only on when the traction power is
  on.
- Add some early design files for the dashboard, body controller and
  remote control.
Parts:
- removed A?: Adafruit_Feather_Generic, Module:Adafruit_Feather, symbol MCU_Module:Adafruit_Feather_Generic
- removed BT? (x2): Battery_Cell, symbol Device:Battery_Cell
- removed BT?: 18650, symbol Device:Battery_Cell
- removed F?: 5V DCDC fuse 5A, symbol Device:Fuse
- removed J? (x5): Conn_01x02, symbol Connector_Generic:Conn_01x02
- removed J?: Outputs, symbol Connector_Generic:Conn_01x08
- removed J? (x3): BNC, symbol Connector_Generic:Conn_01x03
- removed J?: Power, symbol Connector_Generic:Conn_01x02
- removed J?: Relay 1, symbol Connector_Generic:Conn_01x03
- removed J? (x2): XT90, symbol Connector_Generic:Conn_01x02
- removed J?: Conn_01x03, symbol Connector_Generic:Conn_01x03
- removed J?: Inputs, symbol Connector_Generic:Conn_01x08
- removed J?: 12V (XT30), symbol Connector_Generic:Conn_01x02
- removed J?: AT LED, symbol Connector_Generic:Conn_01x02
- removed J? (x3): USB-A socket, symbol Connector_Generic:Conn_01x02
- removed J?: BMS BTN, symbol Connector_Generic:Conn_01x02
- removed J? (x4): Screw_Terminal_01x01, symbol Connector:Screw_Terminal_01x01
- removed J?: Relay 2, symbol Connector_Generic:Conn_01x03
- removed J?: AT CTRLR, symbol Connector:Screw_Terminal_01x01
- removed J?: 1S BMS, symbol Connector_Generic:Conn_02x02_Odd_Even
- removed PS?: DROK 12V-5V Buck, Converter_DCDC:Converter_DCDC_Murata_MEE1SxxxxSC_THT, symbol Converter_DCDC:MEE1S0303SC
- removed SW? (x3): SW_SPST, symbol Switch:SW_SPST
- removed SW?: Keyswitch, symbol Switch:SW_SPST
- removed U?: SSR, Package_SIP:SIP4_Sharp-SSR_P7.62mm_Straight, symbol Relay_SolidState:S102S01
- removed U?: 12V_Boost, symbol enduro-libs:12V_Boost
- added 0V, 84V, J? (x4): Screw_Terminal_01x01, symbol Connector:Screw_Terminal_01x01
- added BT? (x2): Battery, symbol Device:Battery
- added BT?: 18650, symbol Device:Battery_Cell
- added BT? (x2): Battery_Cell, symbol Device:Battery_Cell
- added D?: Antitheft disarmed (red), symbol Device:LED
- added J? (x5): AT CTRLR, symbol Connector_Generic:Conn_01x01
- added J? (x4): AT LED, symbol Connector_Generic:Conn_01x02
- added J? (x2): BMS BTN, symbol Connector_Generic:Conn_01x02
- added J? (x5): Conn_01x02, symbol Connector_Generic:Conn_01x02
- added J? (x2): XT90, symbol Connector_Generic:Conn_01x02
- added J? (x3): 12V (XT30), symbol Connector_Generic:Conn_01x02
- added J?: Relay 1, symbol Connector_Generic:Conn_01x03
- added J?: BNC, symbol Connector_Generic:Conn_01x03
- added J? (x7): USB-A socket, symbol Connector_Generic:Conn_01x02
- added J?: 1S BMS, symbol Connector_Generic:Conn_02x02_Odd_Even
- added J?: CUTOFF, symbol Connector_Generic:Conn_01x02
- added J?: Relay 2, symbol Connector_Generic:Conn_01x03
- added J?: CAv3 8p, symbol Connector_Generic:Conn_01x01
- added J?: Frame NL2 charge socket, symbol Connector:SpeakON_NL2
- added PS?: DROK 12V-5V Buck, Converter_DCDC:Converter_DCDC_Murata_MEE1SxxxxSC_THT, symbol Converter_DCDC:MEE1S0303SC
- added PS?: Buck XW-0885-5-15W-USB 85V in 5V3A out, Converter_DCDC:Converter_DCDC_Murata_MEE1SxxxxSC_THT, symbol Converter_DCDC:MEE1S0303SC
- added R?: 510R, symbol Device:R
- added TP? (x4): TestPoint_Small, symbol Connector:TestPoint_Small
- added U?: AQZ105 SSR RELAY SPST-NO 2.6A 0-100V, Package_SIP:SIP4_Sharp-SSR_P7.62mm_Straight, symbol Relay_SolidState:S102S01
- added U?: SSR, Package_SIP:SIP4_Sharp-SSR_P7.62mm_Straight, symbol Relay_SolidState:S102S01
- added U?: 12V_Boost, symbol enduro-libs:12V_Boost
Connections:
- net Ignition (green) is gone; now on net AT CTRLR: J?.6 (Pin_6)
- net +12V: now also J?.1 (Pin_1), J?.1 (Pin_1), J?.1 (Pin_1), J?.2 (Pin_2), J?.2 (Pin_2); no longer J?.1 (Pin_1)
- net +V (brown): now also J?.1+; no longer J?.1+
- net 12V (red): now also D?.1 (K), D?.1 (K), D?.1 (K), D?.1 (K), D?.1 (K), D?.1 (K), J.1 (Pin_1), J?.1 (Pin_1), J?.1 (Pin_1), J?.1 (Pin_1), J?.1 (Pin_1), J?.1 (Pin_1), J?.1 (Pin_1), J?.1 (Pin_1), J?.1 (Pin_1), J?.1 (Pin_1), J?.1 (Pin_1), J?.1 (Pin_1), J?.1 (Pin_1), J?.1 (Pin_1), J?.1 (Pin_1), J?.1 (Pin_1), J?.1 (Pin_1), J?.1 (Pin_1), J?.1 (Pin_1), J?.1 (Pin_1), J?.1 (Pin_1), J?.2 (Pin_2), J?.2 (Pin_2), J?.2 (Pin_2), J?.2 (Pin_2), J?.2 (Pin_2), J?.3 (Pin_3), J?.3 (Pin_3), J?.3 (Pin_3), J?.3 (Pin_3), J?.3 (Pin_3), J?.8 (Pin_8), PS?.3 (-Vout), SW?.2, TP?.1, U?.4
- net 72V (red): now also BT?.1 (+), J?.1 (Pin_1), J?.1 (Pin_1); no longer BT?.1 (+)
- net AT CTRLR: now also J?.1 (Pin_1)
- net AUX (white): now also J?.2 (Pin_2), J?.2 (Pin_2), J?.2 (Pin_2), U?.4; no longer J?.2 (Pin_2), J?.2 (Pin_2)
- net B+: now also BT?.1 (+), BT?.1 (+), BT?.1 (+), J?.1 (Pin_1)
- net B-: now also BT?.2 (-), BT?.2 (-), BT?.2 (-), J?.3 (Pin_3)
- net DRL (red): now also J?.2 (Pin_2), U?.3; no longer J?.1 (Pin_1), J?.2 (Pin_2)
- net GND (blue): now also J?.1 (Pin_1), PS?.1 (-Vin), J?.1-, PS?.1 (-Vin)
- net NC: now also J?.1 (Pin_1), J?.1 (Pin_1)
- net NO: now also J?.1 (Pin_1), J?.1 (Pin_1), J?.2 (Pin_2), J?.3 (Pin_3), J?.3 (Pin_3); no longer J?.1 (Pin_1), J?.1 (Pin_1)
- net at U?.3: now also J?.1 (Pin_1)
- net at U?.4: now also J?.2 (Pin_2)
- net at BT?.2 (-): now also J?.1 (Pin_1)
- net 84V (red?) renamed Antitheft 84V
- net Antitheft 84V: now also J?.1 (Pin_1), J?.2 (Pin_2); no longer J?.5 (Pin_5)
- removed net Brake12V (red): D?.1 (K), D?.1 (K), D?.1 (K), D?.1 (K), D?.1 (K), D?.1 (K), J.1 (Pin_1), J?.1 (Pin_1), J?.1 (Pin_1), J?.1 (Pin_1), J?.1 (Pin_1), J?.1 (Pin_1), J?.1 (Pin_1), J?.1 (Pin_1), J?.1 (Pin_1), J?.1 (Pin_1), J?.1 (Pin_1), J?.1 (Pin_1), J?.1 (Pin_1), J?.1 (Pin_1), J?.1 (Pin_1), J?.1 (Pin_1), J?.1 (Pin_1), J?.1 (Pin_1), J?.1 (Pin_1), J?.1 (Pin_1), J?.1 (Pin_1), J?.1 (Pin_1), J?.2 (Pin_2), J?.2 (Pin_2), J?.2 (Pin_2), J?.2 (Pin_2), J?.2 (Pin_2), J?.3 (Pin_3), J?.3 (Pin_3), J?.3 (Pin_3), J?.3 (Pin_3), J?.3 (Pin_3), J?.8 (Pin_8), PS?.1 (-Vin), PS?.3 (-Vout), SW?.2
- new net: J?.1 (Pin_1), U?.1
- new net: J?.2 (Pin_2), U?.2
- new net: R?.2, U?.3
- new net: J?.2 (Pin_2), J?.2 (Pin_2), J?.2 (Pin_2), PS?.3 (-Vout)
- new net: J?.1 (Pin_1), J?.1 (Pin_1), J?.1 (Pin_1), PS?.4 (+Vout)
- new net: BT?.2 (-), J?.2 (Pin_2), J?.3 (Pin_3)
- new net: 84V.1 (Pin_1), BT?.1 (+)
- new net: J?.2 (Pin_2), U?. (VOUT-) (x2)
- new net: J?.4 (Pin_4), U?. (VOUT-)
- new net: J?.1 (Pin_1), J?.1 (Pin_1), PS?.4 (+Vout)
- new net: J?.2 (Pin_2), J?.2 (Pin_2), PS?.3 (-Vout)
- new net: J?.1 (Pin_1), U?. (VOUT-)
- new net: J?.2 (Pin_2), R?.1
- new net BATT_0V: J?.1 (Pin_1)
- new net BATT_84V: J?.1 (Pin_1), J?.1 (Pin_1), J?.1+, J?.5 (Pin_5), PS?.2 (+Vin)
- new net COM (yellow): J?.1 (Pin_1), TP?.1, TP?.1
- new net NO (blue): J?.1 (Pin_1), J?.1 (Pin_1), TP?.1
- no-connect marks 10 -> 9
Other:
- added sheet Body Controller (bdc.kicad_sch)
- added sheet Dashboard (dashboard.kicad_sch)
- added sheet Remote (remote.kicad_sch)
- note added: "1.5V max drop across LED ~7mA forward current 3mA required"
- note added: "5V STANDBY JST"
- note added: "5VSB USB-A"
- note added: "84V (red?)"
- note added: "BMS BTN"
- note added: "GND (black)"
- note added: "JBD BMS 200A continuous"
- note added: "Junkyard"
- note added: "Mounted on side case. Antitheft LED stays lit even if the cutoff is open. It's your reminder to lock the bike before walking away."
- note added: "OUT+"
- note added: "OUT-"
- note added: "RPi Dashboard"
- note added: "Remote module Assembled on protoboard"
- note added: "SMART ANT BMS 120A continuous"
- note added: "The GNDs are NOT isolated Supply is ALWAYS ON. To disable, switch off the BMS discharge FET. Always on. BDC and remote receiver only."
- note added: "revise"
- note added: "spare for body controller"
- note added: "todo"
- note removed: "12VSB charger"
- note removed: "Antitheft line to controller and CAv3"
- note removed: "CAv3 orange line Sabvoton antitheft/orange line Put remote alarm in series"
- note removed: "CT-22 Display"
- note removed: "Cutoff/Killswitch Relay"
- note removed: "Flipsky antispark 150A"
- note removed: "Hilitand MOS FET PWM 3-20V to 3.7-27VDC 10A 4-Channel Driver Module PLC Amplifier Circuit Board"
- note removed: "NOYITO Isolated MOS FET Field Effect Transistor Module Optocoupler isolation Alternative Relay FR120N 100V 9.4A"
- note removed: "TODO remove flipsky"
- note removed: "UP TO HERE CAV3 orange and Sabvoton ignition both go to bullet connector which connects back to SSR -OUT"
- note removed: "We want a FET here because we're switching 84V on the secondary. Relays that can do that are large and expensive."
